Commit message: added mapping with octo and launch raspberry cam

File: turtlebot3_description/urdf/turtlebot3_radar_burger.urdf.xacro (robot description, xacro)
@@ -116,16 +116,34 @@
     <parent link="base_link"/>
     <child link="ti_mmwave"/>
-    <origin xyz="-0.032 0 0.172" rpy="0 0 0"/>
+    <origin xyz="0.05 0 0.120" rpy="0 0 0"/>
   </joint>
   <link name="ti_mmwave">
     <origin xyz="0 0 0.0" rpy="0 0 0"/>
     <collision>
-      <origin xyz="0.015 0 -0.0065" rpy="0 0 0"/>
+      <origin xyz="0.000 0 0.035" rpy="0 0 0"/>
       <geometry>
-        <cylinder length="0.0315" radius="0.055"/>
+        <box size="0.0150 0.080 0.090"/>
       </geometry>
+      <material name="Cyan">
+         <color rgba="0 1.0 1.0 1.0"/>
+      </material>
     </collision>
     <inertial>
-      <mass value="0.05" />
+      <mass value="0.005" />
+      <origin xyz="0 0 0" />
+      <inertia ixx="0.001" ixy="0.0" ixz="0.0"
+               iyy="0.001" iyz="0.0"
+               izz="0.001" />
+    </inertial>
+  </link>
+  <joint name="radar_cam_joint" type="fixed">
+    <parent link="base_link"/>
+    <child link="rasp_cam_frame"/>
+    <origin xyz="0.05 0 0.21" rpy="0 0 0"/>
+  </joint>
+  <link name="rasp_cam_frame">
+    <origin xyz="0 0 0.0" rpy="0 0 0"/>
+    <inertial>
+      <mass value="0.005" />
       <origin xyz="0 0 0" />
       <inertia ixx="0.001" ixy="0.0" ixz="0.0"

Commit message: Change real locations ca radar and launch separately

File: turtlebot3_description/urdf/turtlebot3_radar_burger.urdf.xacro (robot description, xacro)
@@ -115,8 +115,8 @@
   <joint name="scan_joint" type="fixed">
     <parent link="base_link"/>
-    <child link="ti_mmwave"/>
-    <origin xyz="0.05 0 0.120" rpy="0 0 0"/>
+    <child link="ti_mmwave_frame"/>
+    <origin xyz="0.025 0 0.1" rpy="0 0 0"/>
   </joint>
-  <link name="ti_mmwave">
+  <link name="ti_mmwave_frame">
     <origin xyz="0 0 0.0" rpy="0 0 0"/>
     <collision>
@@ -140,8 +140,8 @@
     <parent link="base_link"/>
     <child link="rasp_cam_frame"/>
-    <origin xyz="0.05 0 0.21" rpy="0 0 0"/>
+    <origin xyz="0.017 0 0.205" rpy="0 0 0"/>
   </joint>
   <link name="rasp_cam_frame">
-    <origin xyz="0 0 0.0" rpy="0 0 0"/>
+    <origin xyz="0.003 0.01 -0.0105" rpy="0 0 0"/>
     <inertial>
       <mass value="0.005" />

Commit message: new limits

File: turtlebot3_description/urdf/turtlebot3_radar_burger.urdf.xacro (robot description, xacro)
@@ -116,8 +116,8 @@
     <parent link="base_link"/>
     <child link="ti_mmwave_frame"/>
-    <origin xyz="0.025 0 0.1" rpy="0 0 0"/>
+    <origin xyz="0.045 0.02 0.125" rpy="0 0 0"/>
   </joint>
   <link name="ti_mmwave_frame">
-    <origin xyz="0 0 0.0" rpy="0 0 0"/>
+    <origin xyz="0 -0.01 0.02" rpy="0 0 0"/>
     <collision>
       <origin xyz="0.000 0 0.035" rpy="0 0 0"/>
@@ -137,11 +137,11 @@
     </inertial>
   </link>
-  <joint name="radar_cam_joint" type="fixed">
+  <joint name="cam_joint" type="fixed">
     <parent link="base_link"/>
     <child link="rasp_cam_frame"/>
-    <origin xyz="0.017 0 0.205" rpy="0 0 0"/>
+    <origin xyz="0.025 0.0 0.175" rpy="0 0 0"/>
   </joint>
   <link name="rasp_cam_frame">
-    <origin xyz="0.003 0.01 -0.0105" rpy="0 0 0"/>
+    <origin xyz="0.020 0 0.0105" rpy="0 0 0"/>
     <inertial>
       <mass value="0.005" />

Commit message: New turtlebot_radar package from TI reduced ros driver

File: turtlebot3_description/urdf/turtlebot3_radar_burger.urdf.xacro (robot description, xacro)
@@ -3,4 +3,7 @@
   <xacro:include filename="$(find turtlebot3_description)/urdf/common_properties.xacro"/>
   <xacro:include filename="$(find turtlebot3_description)/urdf/turtlebot3_burger.gazebo.xacro"/>
+  <material name="red">
+    <color rgba="1 0 0 1"/>
+  </material>
   <link name="base_footprint"/>
   <joint name="base_joint" type="fixed">
@@ -129,11 +132,10 @@
       </material>
     </collision>
-    <inertial>
-      <mass value="0.005" />
-      <origin xyz="0 0 0" />
-      <inertia ixx="0.001" ixy="0.0" ixz="0.0"
-               iyy="0.001" iyz="0.0"
-               izz="0.001" />
-    </inertial>
+   <visual>
+        <geometry>
+          <box size="0.01 0.05 0.06" />
+        </geometry>
+        <material name="red"/>
+      </visual>
   </link>
   <joint name="cam_joint" type="fixed">

Commit message: change levels of azimuth and elevation radar

File: turtlebot3_description/urdf/turtlebot3_radar_burger.urdf.xacro (robot description, xacro)
@@ -3,7 +3,4 @@
   <xacro:include filename="$(find turtlebot3_description)/urdf/common_properties.xacro"/>
   <xacro:include filename="$(find turtlebot3_description)/urdf/turtlebot3_burger.gazebo.xacro"/>
-  <material name="red">
-    <color rgba="1 0 0 1"/>
-  </material>
   <link name="base_footprint"/>
   <joint name="base_joint" type="fixed">
@@ -119,8 +116,8 @@
     <parent link="base_link"/>
     <child link="ti_mmwave_frame"/>
-    <origin xyz="0.045 0.02 0.125" rpy="0 0 0"/>
+    <origin xyz="0.057 0.01 0.14" rpy="0 0 0"/>
   </joint>
   <link name="ti_mmwave_frame">
-    <origin xyz="0 -0.01 0.02" rpy="0 0 0"/>
+    <origin xyz="0 0 0" rpy="0 0 0"/>
     <collision>
       <origin xyz="0.000 0 0.035" rpy="0 0 0"/>
@@ -132,18 +129,12 @@
       </material>
     </collision>
-   <visual>
-        <geometry>
-          <box size="0.01 0.05 0.06" />
-        </geometry>
-        <material name="red"/>
-      </visual>
   </link>
   <joint name="cam_joint" type="fixed">
     <parent link="base_link"/>
     <child link="rasp_cam_frame"/>
-    <origin xyz="0.025 0.0 0.175" rpy="0 0 0"/>
+    <origin xyz="0.052 0.0 0.185" rpy="0 0 0"/>
   </joint>
   <link name="rasp_cam_frame">
-    <origin xyz="0.020 0 0.0105" rpy="0 0 0"/>
+    <origin xyz="0.0 0 0" rpy="0 0 0"/>
     <inertial>
       <mass value="0.005" />

Commit message: change axis for camera optical frame

File: turtlebot3_description/urdf/turtlebot3_radar_burger.urdf.xacro (robot description, xacro)
@@ -133,5 +133,5 @@
     <parent link="base_link"/>
     <child link="rasp_cam_frame"/>
-    <origin xyz="0.052 0.0 0.185" rpy="0 0 0"/>
+    <origin xyz="0.052 0.0 0.185" rpy="-1.57079632679 0 -1.57079632679"/>
   </joint>
   <link name="rasp_cam_frame">

Commit message: Adap optical frame axis

File: turtlebot3_description/urdf/turtlebot3_radar_burger.urdf.xacro (robot description, xacro)
@@ -133,5 +133,5 @@
     <parent link="base_link"/>
     <child link="rasp_cam_frame"/>
-    <origin xyz="0.052 0.0 0.185" rpy="-1.57079632679 0 -1.57079632679"/>
+    <origin xyz="0.052 0.0 0.185" rpy="1.57079632679 0 -1.57079632679"/>
   </joint>
   <link name="rasp_cam_frame">

Commit message: corerct axis values

File: turtlebot3_description/urdf/turtlebot3_radar_burger.urdf.xacro (robot description, xacro)
@@ -133,5 +133,5 @@
     <parent link="base_link"/>
     <child link="rasp_cam_frame"/>
-    <origin xyz="0.052 0.0 0.185" rpy="1.57079632679 0 -1.57079632679"/>
+    <origin xyz="0.052 0.0 0.185" rpy="-1.57079632679 0 1.57079632679"/>
   </joint>
   <link name="rasp_cam_frame">

Commit message: fixed rotation optical frame

File: turtlebot3_description/urdf/turtlebot3_radar_burger.urdf.xacro (robot description, xacro)
@@ -130,8 +130,9 @@
     </collision>
   </link>
+yaw, pitch, and roll about Z, Y, X
   <joint name="cam_joint" type="fixed">
     <parent link="base_link"/>
     <child link="rasp_cam_frame"/>
-    <origin xyz="0.052 0.0 0.185" rpy="-1.57079632679 0 1.57079632679"/>
+    <origin xyz="0.052 0.0 0.185" rpy="0 1.57079632679 0"/>
   </joint>
   <link name="rasp_cam_frame">
